Commit message: removing shifting creataing bins

File: src/hrwros_support/urdf/hrwros.xacro (robot description, xacro)
@@ -20,8 +20,4 @@
   <xacro:include filename="$(find hrwros_support)/urdf/bin/bin.urdf.xacro"/>
   <xacro:bin_urdf prefix="bin_1_"/>
-  <xacro:bin_urdf prefix="bin_2_"/>
-  <xacro:bin_urdf prefix="bin_3_"/>
-  <xacro:bin_urdf prefix="bin_4_"/>
-  <xacro:bin_urdf prefix="bin_5_"/>
   <!-- Joints -->
   <joint name="world_interface_to_world" type="fixed">
@@ -50,29 +46,16 @@
     <parent link="world_interface" />
     <child link="bin_1_base_link" />
-    <origin xyz="-0.3 1.2 0.0" rpy="0 0 0" />
+    <origin xyz="-8.0 -2.2 0.0" rpy="0 0 0" />
   </joint>
-  <!-- bin 2 -->
-  <joint name="bin_2_joint" type="fixed">
-    <parent link="world_interface" />
-    <child link="bin_2_base_link" />
-    <origin xyz="-0.3 0.4 0.0" rpy="0 0 0" />
-  </joint>
-  <!-- bin 3 -->
-  <joint name="bin_3_joint" type="fixed">
-    <parent link="world_interface" />
-    <child link="bin_3_base_link" />
-    <origin xyz="-0.3 -0.4 0.0" rpy="0 0 0" />
-  </joint>
-  <!-- bin 4 -->
-  <joint name="bin_4_joint" type="fixed">
-    <parent link="world_interface" />
-    <child link="bin_4_base_link" />
-    <origin xyz="-0.3 -1.2 0.0" rpy="0 0 0" />
-  </joint>
-  <!-- bin 5 -->
-  <joint name="bin_5_joint" type="fixed">
-    <parent link="world_interface" />
-    <child link="bin_5_base_link" />
-    <origin xyz="-0.3 -2.0 0.0" rpy="0 0 0" />
-  </joint>
+ <link name="robot2_pedestral_link">
+  <visual>
+    <geometry>
+     <box size="1 1 1" />
+    </geometry>
+  </visual>
+ </link>
+ <joint name="robo2_pedestal_joint" type="fixed">
+  <parent link="world"/>
+  <child link="robot2_pedestral_link" />
+</joint>
 </robot>

Commit message: adding a box with color and material

File: src/hrwros_support/urdf/hrwros.xacro (robot description, xacro)
@@ -50,7 +50,11 @@
  <link name="robot2_pedestral_link">
   <visual>
+   <origin xyz="0 0 0.3"/>
     <geometry>
-     <box size="1 1 1" />
+     <box size = "0.3 0.3 0.6"/>
     </geometry>
+    <material name= 'robot2_pedestal_color'>
+     <color rgba="0 0.16 0.53 1"/>
+    </material>
   </visual>
  </link>

Commit message: changing the origin for the box

File: src/hrwros_support/urdf/hrwros.xacro (robot description, xacro)
@@ -62,4 +62,5 @@
   <parent link="world"/>
   <child link="robot2_pedestral_link" />
+  <origin xyz="-7.8 -1.5 0"/>
 </joint>
 </robot>

Commit message: adding the robot using xacro file in the environment

File: src/hrwros_support/urdf/hrwros.xacro (robot description, xacro)
@@ -48,5 +48,5 @@
     <origin xyz="-8.0 -2.2 0.0" rpy="0 0 0" />
   </joint>
- <link name="robot2_pedestral_link">
+ <link name="robot2_pedestal_link">
   <visual>
    <origin xyz="0 0 0.3"/>
@@ -61,6 +61,13 @@
  <joint name="robo2_pedestal_joint" type="fixed">
   <parent link="world"/>
-  <child link="robot2_pedestral_link" />
+  <child link="robot2_pedestal_link" />
   <origin xyz="-7.8 -1.5 0"/>
-</joint>
+ </joint>
+<xacro:include filename="$(find ur_description)/urdf/ur5.urdf.xacro"/>
+<xacro:ur5_robot prefix="robot2_" joint_limited="true"/>
+ <joint name="robot2-robot2_pedestal_joint" type="fixed">
+  <parent link="robot2_pedestal_link"/>
+  <child link="robot2_base_link"/>
+  <origin xyz="0 0 0.6" rpy="0 0 ${radians(90)}"/>
+ </joint>
 </robot>

Commit message: setup for week3 autonautonomous robots

File: src/hrwros_support/urdf/hrwros.xacro (robot description, xacro)
@@ -17,7 +17,31 @@
   <xacro:include filename="$(find hrwros_support)/urdf/vacuum_gripper/vacuum_gripper.urdf.xacro"/>
   <xacro:vacuum_gripper_urdf prefix="vacuum_gripper1_" joint_prefix="vacuum_gripper1_joint"/>
+  <!-- Robot2 Pedestal -->
+  <xacro:include filename="$(find hrwros_support)/urdf/robot_pedestal/robot_pedestal.urdf.xacro"/>
+  <xacro:robot_pedestal_urdf pedestal_prefix="robot2_" pedestal_parent="world_interface" pedestal_height="0.7">
+    <origin xyz="-7.8 -1.5 0.0" rpy="0 0 0"/>
+  </xacro:robot_pedestal_urdf>
+  <!-- Robot2 -->
+  <xacro:include filename="$(find ur_description)/urdf/ur5.urdf.xacro"/>
+  <xacro:ur5_robot prefix="robot2_" joint_limited="true"/>
+  <!-- Vacuum Gripper2 -->
+  <xacro:include filename="$(find hrwros_support)/urdf/vacuum_gripper/vacuum_gripper.urdf.xacro"/>
+  <xacro:vacuum_gripper_urdf prefix="vacuum_gripper2_" joint_prefix="vacuum_gripper2_joint"/>
   <!-- bins -->
   <xacro:include filename="$(find hrwros_support)/urdf/bin/bin.urdf.xacro"/>
   <xacro:bin_urdf prefix="bin_1_"/>
+  <!-- logical camera 1 collision model -->
+  <xacro:include filename="$(find hrwros_support)/urdf/logical_camera/logical_camera.urdf.xacro"/>
+  <xacro:logical_camera_urdf prefix="logical_camera1_" logical_camera_parent="world_interface">
+    <origin xyz="1.2 1.8 2.0" rpy="0 1.5708 0"/>
+  </xacro:logical_camera_urdf>
+  <!-- logical camera 2 collision model -->
+  <xacro:include filename="$(find hrwros_support)/urdf/logical_camera/logical_camera.urdf.xacro"/>
+  <xacro:logical_camera_urdf prefix="logical_camera2_" logical_camera_parent="world_interface">
+    <origin xyz="-8.3 -1.23 1.8" rpy="0 1.5708 0"/>
+  </xacro:logical_camera_urdf>
+  <!-- break beam -->
+  <xacro:include filename="$(find hrwros_support)/urdf/break_beam/break_beam.urdf.xacro"/>
+  <xacro:break_beam_urdf prefix="break_beam_"/>
   <!-- Joints -->
   <joint name="world_interface_to_world" type="fixed">
@@ -33,6 +57,6 @@
   <!-- robot1 to pedestal. -->
   <joint name="robot1_to_pedestal" type="fixed">
-  <origin xyz="0 0 0.95" rpy="0 0 0" />
-  <parent link="robot1_pedestal_link" />
+  <origin xyz="0.5 1.8 0.95" rpy="0 0 0" />
+  <parent link="world_interface" />
   <child link="robot1_base_link" />
   </joint>
@@ -42,5 +66,27 @@
     <child link="vacuum_gripper1_base_link" />
   </joint>
-  <!-- bin 1 -->
+  <!-- robot2-pedestal to world. -->
+  <joint name="robot2_pedestal_to_world_interface" type="fixed">
+    <parent link="world_interface" />
+    <child link="robot2_pedestal_link" />
+    <origin xyz="-7.8 -1.5 0.0" rpy="0.0 0.0 0.0"/>
+  </joint>
+  <!-- robot2 to pedestal. -->
+  <joint name="robot2_to_pedestal" type="fixed">
+    <parent link="world_interface" />
+    <child link="robot2_base_link" />
+    <origin xyz="-7.8 -1.5 0.7" rpy="0 0 1.57" />
+  </joint>
+  <!-- gripper2 to robot2. -->
+  <joint name="gripper2_to_robot2" type="fixed">
+    <parent link="robot2_tool0" />
+    <child link="vacuum_gripper2_base_link" />
+  </joint>
+  <!-- break beam to world. -->
+  <joint name="break_beam_joint" type="fixed">
+    <parent link="world_interface" />
+    <child link="break_beam_world_interface" />
+  </joint>
+  <!-- bin to world. -->
   <joint name="bin_1_joint" type="fixed">
     <parent link="world_interface" />
@@ -48,26 +94,3 @@
     <origin xyz="-8.0 -2.2 0.0" rpy="0 0 0" />
   </joint>
- <link name="robot2_pedestal_link">
-  <visual>
-   <origin xyz="0 0 0.3"/>
-    <geometry>
-     <box size = "0.3 0.3 0.6"/>
-    </geometry>
-    <material name= 'robot2_pedestal_color'>
-     <color rgba="0 0.16 0.53 1"/>
-    </material>
-  </visual>
- </link>
- <joint name="robo2_pedestal_joint" type="fixed">
-  <parent link="world"/>
-  <child link="robot2_pedestal_link" />
-  <origin xyz="-7.8 -1.5 0"/>
- </joint>
-<xacro:include filename="$(find ur_description)/urdf/ur5.urdf.xacro"/>
-<xacro:ur5_robot prefix="robot2_" joint_limited="true"/>
- <joint name="robot2-robot2_pedestal_joint" type="fixed">
-  <parent link="robot2_pedestal_link"/>
-  <child link="robot2_base_link"/>
-  <origin xyz="0 0 0.6" rpy="0 0 ${radians(90)}"/>
- </joint>
 </robot>
